File: pcb/usb_c_cable_tester.kicad_pcb (KiCad board)
At the start: 2 copper layers, 85.6 x 54 mm, 60 parts, among them J1 USB_C_Receptacle, J2 USB_C_Receptacle_ALLPINS, J3 USB_B_Micro, J4 USB3_B, J5 USB_B_Mini, J6 USB3_A

Commit message: changes (and a bit chaos)
Parts:
- moved J3 0.30 mm to (139.8, 97.0)
Routing:
- net GND: track 32.9 -> 49.3 mm, vias 27 -> 30
